File: environment-sensor.kicad_sch (KiCad schematic)
At the start: 109 parts, among them J1 USB-C_GCT_USB4105-GF-A, J2 JST_SH_1x4_SM04B-SRSS-TB-LF-SN, J3 JST_SH_1x4_SM04B-SRSS-TB-LF-SN, U1 FT232R_QFN, U2 AP7370-33SA-7, U3 STM32G474CET6, U4 MB85RC1MTPNF-G, U5 SHT45, U6 BME280, Y1 Resonator_32.768kHz_ECX-31B, Y2 Resonator_8MHz_ABM3B

Commit message: [#60742] Add updated components
Parts:
- C1, C10, C11, C12, C13, C14, C15, C16, C17, C18, C19, C2, C20, C21, C22, C23, C24, C25, C26, C27, C28, C3, C4, C5, C6, C7, C8, C9, D1, D2, D3, D4, D7, D9, FB1, FB2, FB3, LD1, LD2, MP1, MP2, MP3, N1, N2, R1, R10, R11, R12, R13, R14, R15, R16, R17, R18, R19, R2, R20, R21, R22, R23, R24, R25, R26, R27, R28, R29, R3, R30, R31, R32, R33, R34, R35, R36, R37, R38, R4, R5, R6, R7, R8, R9, TP1, TP10, TP11, TP12, TP2, TP3, TP4, TP5, TP6, TP7, TP8, TP9, Y1, Y2: Public (none) -> False
Connections:
- no-connect marks 34 -> 32
